Commit message: Add gazebo_control , rsp_sim.launch.py and the package teleop

File: description/robot.urdf.xacro (robot description, xacro)
@@ -2,3 +2,4 @@
 <robot xmlns:xacro="http://www.ros.org/wiki/xacro"  name="robot">
     <xacro:include filename = "robot_core.xacro" />
+    <xacro:include filename = "gazebo_control.xacro"/>
 </robot>

File: description/robot_core.xacro (robot description, xacro)
@@ -1,111 +1,125 @@
 <?xml version="1.0"?>
-<robot xmlns:xacro="http://www.ros.org/wiki/xacro">
-    <xacro:include filename = "inertial_macros.xacro"/>
-    <material name = "white">
-        <color rgba = "1 1 1 1"/>
+<robot xmlns:xacro="http://www.ros.org/wiki/xacro" >
+    <xacro:include filename="inertial_macros.xacro"/>
+    <material name="white">
+        <color rgba="1 1 1 1" />
     </material>
-    <material name = "orange">
-        <color rgba = "1 0.3 0.1 1"/>
+    <material name="orange">
+        <color rgba="1 0.3 0.1 1"/>
     </material>
-    <material name = "blue">
-    <color rgba = "0.2 0.2 1 1"/>
+    <material name="blue">
+        <color rgba="0.2 0.2 1 1"/>
     </material>
-    <material name = "black">
-        <color rgba = "0 0 0 1"/>
+    <material name="black">
+        <color rgba="0 0 0 1"/>
     </material>
     <!-- BASE LINK -->
-    <link name = "base_link">
+    <link name="base_link">
     </link>
     <!-- CHASSIS LINK -->
-    <joint name = "chassis_joint" type = "fixed">
-        <parent link = "base_link"/>
-        <child link = "chassis"/>
-        <origin xyz = "-0.1 0 0"/>
+    <joint name="chassis_joint" type="fixed">
+        <parent link="base_link"/>
+        <child link="chassis"/>
+        <origin xyz="-0.1 0 0"/>
     </joint>
-    <link name = "chassis">
+    <link name="chassis">
         <visual>
-            <origin xyx = "0.15 0 0.075"/>
+            <origin xyz="0.15 0 0.075"/>
             <geometry>
-                <box size = "0.3 0.3 0.15"/>
+                <box size="0.3 0.3 0.15"/>
             </geometry>
-            <material name = "white"/>
+            <material name="white"/>
         </visual>
-        <colision>
-            <origin xyx = "0.15 0 0.075"/>
+        <collision>
+            <origin xyz="0.15 0 0.075"/>
             <geometry>
-                <box size = "0.3 0.3 0.15"/>
+                <box size="0.3 0.3 0.15"/>
             </geometry>
-        </colision>
-        <xacro:inertial_box mass = "0.5" x = "0.3" y = "0.3" z = "0.15">
-            <origin xyz = "0.15 0 0.075" rpy = "0 0 0"/>
+        </collision>
+        <xacro:inertial_box mass="0.5" x="0.3" y="0.3" z="0.15">
+            <origin xyz="0.15 0 0.075" rpy="0 0 0"/>
         </xacro:inertial_box>
     </link>
+    <gazebo reference="chassis">
+        <material>Gazebo/White</material>
+    </gazebo>
     <!-- LEFT WHEEL LINK -->
-    <joint name = "left_wheel_joint" type = "continuous">
-        <parent link = "base_link"/>
-        <child link = "left_wheel"/>
-        <origin xyz = "0 0.175 0" rpy = "-${pi/2} 0 0"/>
-        <axis xyz = "0 0 1"/>
+    <joint name="left_wheel_joint" type="continuous">
+        <parent link="base_link"/>
+        <child link="left_wheel"/>
+        <origin xyz="0 0.175 0" rpy="-${pi/2} 0 0" />
+        <axis xyz="0 0 1"/>
     </joint>
-    <link name = "left_wheel">
+    <link name="left_wheel">
         <visual>
             <geometry>
-                <cylinder radius = "0.05" length = "0.04"/>
+                <cylinder radius="0.05" length="0.04"/>
             </geometry>
-            <material name = "blue"/>
+            <material name="blue"/>
         </visual>
-        <colision>
+        <collision>
             <geometry>
-                <cylinder radius = "0.05" length = "0.04"/>
+                <cylinder radius="0.05" length="0.04"/>
             </geometry>
-        </colision>
-        <xacro:inertial_cylinder mass = "0.1" length = "0.04" radius = "0.05">
-            <origin xyz = "0 0 0" rpy = "0 0 0"/>
+        </collision>
+        <xacro:inertial_cylinder mass="0.1" length="0.04" radius="0.05">
+            <origin xyz="0 0 0" rpy="0 0 0"/>
         </xacro:inertial_cylinder>
     </link>
-    <!--RIGHT WHEEL LINK -->
-    <joint name = "right_wheel_joint" type = "continuous">
-        <parent link = "base_link"/>
-        <child link = "right_wheel"/>
-        <origin xyz = "0 -0.175 0" rpy = "${pi/2} 0 0"/>
-        <axis xyz = "0 0 -1"/>
+    <gazebo reference="left_wheel">
+        <material>Gazebo/Blue</material>
+    </gazebo>
+    <!-- RIGHT WHEEL LINK -->
+    <joint name="right_wheel_joint" type="continuous">
+        <parent link="base_link"/>
+        <child link="right_wheel"/>
+        <origin xyz="0 -0.175 0" rpy="${pi/2} 0 0" />
+        <axis xyz="0 0 -1"/>
     </joint>
-    <link name = "right_wheel">
+    <link name="right_wheel">
         <visual>
             <geometry>
-                <cylinder radius = "0.05" length = "0.04"/>
+                <cylinder radius="0.05" length="0.04"/>
             </geometry>
-            <material name = "blue"/>
+            <material name="blue"/>
         </visual>
-        <colision>
+        <collision>
             <geometry>
-                <cylinder radius = "0.05" length = "0.04"/>
+                <cylinder radius="0.05" length="0.04"/>
             </geometry>
-        </colision>
-        <xacro:inertial_cylinder mass = "0.1" length = "0.04" radius = "0.05">
-            <origin xyz = "0 0 0" rpy = "0 0 0"/>
+        </collision>
+        <xacro:inertial_cylinder mass="0.1" length="0.04" radius="0.05">
+            <origin xyz="0 0 0" rpy="0 0 0"/>
         </xacro:inertial_cylinder>
     </link>
+    <gazebo reference="right_wheel">
+        <material>Gazebo/Blue</material>
+    </gazebo>
     <!-- CASTER WHEEL LINK -->
-    <joint name = "caster_wheel" type = "fixed">
-        <parent link = "chassis"/>
-        <child link = "caster_wheel"/>
-        <origin xyz = "-0.1 0 -0.08"/>
+    <joint name="caster_wheel_joint" type="fixed">
+        <parent link="chassis"/>
+        <child link="caster_wheel"/>
+        <origin xyz="0.24 0 0"/>
     </joint>
-    <link name = "caster_wheel">
+    <link name="caster_wheel">
         <visual>
             <geometry>
-                <sphere radius = "0.05"/>
+                <sphere radius="0.05"/>
             </geometry>
-            <material name = "black"/>
+            <material name="black"/>
         </visual>
-        <colision>
+        <collision>
             <geometry>
-                <sphere radius = "0.05"/>
+                <sphere radius="0.05"/>
             </geometry>
-        </colision>
-        <xacro:inertial_sphere mass = "0.1" radius = "0.05">
-            <origin xyz = "0 0 0" rpy = "0 0 0"/>
+        </collision>
+        <xacro:inertial_sphere mass="0.1" radius="0.05">
+            <origin xyz="0 0 0" rpy="0 0 0"/>
         </xacro:inertial_sphere>
     </link>
+    <gazebo reference="caster_wheel">
+        <material>Gazebo/Black</material>
+        <mu1 value="0.001"/>
+        <mu2 value="0.001"/>
+    </gazebo>
 </robot>
